Commit message: added simple planning interface

File: aubo_i5_description/urdf/aubo_i5.xacro (robot description, xacro)
@@ -10,4 +10,5 @@
     hw_interface="$(arg transmission_hw_interface)"
     parent="world"
+    tcp_offset="0"
   >
     <origin xyz="0 0 0" rpy="0 0 0" />

File: aubo_i5_description/urdf/aubo_i5_macro.xacro (robot description, xacro)
@@ -8,4 +8,5 @@
     parent
     hw_interface
+    tcp_offset
     *origin"
   >
@@ -164,4 +165,6 @@
       </collision>
     </link>
+    <link name="${prefix}tool0_link"/>
+    <link name="${prefix}tcp_link"/>
     <joint name="${prefix}base_joint" type="fixed">
       <parent link="${parent}" />
@@ -217,4 +220,14 @@
         effort="${max_effort_2}" />
     </joint>
+    <joint name="${prefix}tool0_joint" type="fixed">
+      <parent link="${prefix}wrist_3_link" />
+      <child link="${prefix}tool0_link" />
+      <origin xyz="0.0 -0.0335 0.0" rpy="${pi/2} 0 0" />
+    </joint>
+    <joint name="${prefix}tcp_joint" type="fixed">
+      <parent link="${prefix}tool0_link" />
+      <child link="${prefix}tcp_link" />
+      <origin xyz="0.0 0.0 ${tcp_offset}" rpy="${-pi} 0 ${pi/2}" />
+    </joint>
   </xacro:macro>
 </robot>

File: aubo_i5_moveit_config/config/gazebo_aubo_i5.urdf (robot description, URDF)
Before this commit: robot aubo_i5, 8 links, 7 joints
Links:
- added link tcp_link
- added link tool0_link
Joints:
- added joint tcp_joint: type fixed, parent tool0_link, child tcp_link, origin xyz=0.0 0.0 0 rpy=-3.141592653589793 0 1.5707963267948966
- added joint tool0_joint: type fixed, parent wrist_3_link, child tool0_link, origin xyz=0.0 -0.0335 0.0 rpy=1.5707963267948966 0 0
