Commit message: moveit working

File: aubo_i5_description/urdf/aubo_i5_macro.xacro (robot description, xacro)
@@ -1,19 +1,14 @@
 <?xml version="1.0"?>
 <robot name="aubo_i5_macro" xmlns:xacro="http://www.ros.org/wiki/xacro">
-  <xacro:include filename="$(find aubo_i5_description)/urdf/aubo_i5_transmission.xacro" />
-  <xacro:include filename="$(find aubo_i5_description)/urdf/aubo_i5_gazebo.xacro" />
   <xacro:macro name="aubo_i5"
     params="
     prefix
     parent
-    hw_interface
     tcp_offset
     *origin"
   >
-    <xacro:aubo_i5_transmission prefix="${prefix}" hw_interface="${hw_interface}" />
-    <xacro:aubo_i5_gazebo prefix="${prefix}" />
     <xacro:property name="lower_limit" value="-3.04" />
     <xacro:property name="upper_limit" value="3.04" />
-    <xacro:property name="max_velocity" value="${pi}" />
+    <xacro:property name="max_velocity" value="3.1" />
     <xacro:property name="max_effort_1" value="300.0" />
     <xacro:property name="max_effort_2" value="50.0" />

File: aubo_i5_moveit_config/config/aubo_i5.urdf.xacro (robot description, xacro)
@@ -3,5 +3,5 @@
     <xacro:arg name="initial_positions_file" default="initial_positions.yaml" />
     <!-- Import aubo_i5 urdf file -->
-    <xacro:include filename="$(find aubo_i5_description)/urdf/aubo_i5.xacro" />
+    <xacro:include filename="$(find aubo_i5_description)/urdf/aubo_i5.urdf.xacro" />
     <!-- Import control_xacro -->
     <xacro:include filename="aubo_i5.ros2_control.xacro" />

Commit message: change base_link name

File: aubo_i5_description/urdf/aubo_i5_macro.xacro (robot description, xacro)
@@ -13,5 +13,5 @@
     <xacro:property name="max_effort_1" value="300.0" />
     <xacro:property name="max_effort_2" value="50.0" />
-    <link name="${prefix}base_link">
+    <link name="${prefix}aubo_i5_base_link">
       <inertial>
         <origin xyz="5.280333978763784e-09 0.0015966894220128586 0.016570455971104445" rpy="0 0 0" />
@@ -164,10 +164,10 @@
     <joint name="${prefix}base_joint" type="fixed">
       <parent link="${parent}" />
-      <child link="${prefix}base_link" />
+      <child link="${prefix}aubo_i5_base_link" />
       <xacro:insert_block name="origin" />
     </joint>
     <joint name="${prefix}shoulder_pan_joint" type="revolute">
       <origin xyz="0.0 0.0 0.0435" rpy="0 0 0" />
-      <parent link="${prefix}base_link" />
+      <parent link="${prefix}aubo_i5_base_link" />
       <child link="${prefix}shoulder_link" />
       <axis xyz="-0.0 0.0 1.0" />
