Commit message: added velocity state interface and compliance controller

File: aubo_driver/urdf/aubo.ros2_control.xacro (robot description, xacro)
@@ -27,4 +27,5 @@
         </command_interface>
         <state_interface name="position"/>
+        <state_interface name="velocity"/>
       </joint>
       <joint name="${prefix}shoulder_lift_joint">
@@ -34,4 +35,5 @@
         </command_interface>
         <state_interface name="position"/>
+        <state_interface name="velocity"/>
       </joint>
       <joint name="${prefix}elbow_joint">
@@ -41,4 +43,5 @@
         </command_interface>
         <state_interface name="position"/>
+        <state_interface name="velocity"/>
       </joint>
       <joint name="${prefix}wrist_1_joint">
@@ -48,4 +51,5 @@
         </command_interface>
         <state_interface name="position"/>
+        <state_interface name="velocity"/>
       </joint>
       <joint name="${prefix}wrist_2_joint">
@@ -55,4 +59,5 @@
         </command_interface>
         <state_interface name="position"/>
+        <state_interface name="velocity"/>
       </joint>
       <joint name="${prefix}wrist_3_joint">
@@ -62,4 +67,5 @@
         </command_interface>
         <state_interface name="position"/>
+        <state_interface name="velocity"/>
       </joint>
     </ros2_control>

File: aubo_i5_description/urdf/aubo_i5.urdf.xacro (robot description, xacro)
@@ -12,5 +12,4 @@
     prefix="$(arg prefix)"
     parent="world"
-    tcp_offset="0"
   >
     <origin xyz="0 0 0" rpy="0 0 0" />

File: aubo_i5_description/urdf/aubo_i5_macro.xacro (robot description, xacro)
@@ -5,5 +5,4 @@
     prefix
     parent
-    tcp_offset
     *origin"
   >
@@ -161,5 +160,4 @@
     </link>
     <link name="${prefix}tool0_link"/>
-    <link name="${prefix}tcp_link"/>
     <joint name="${prefix}base_joint" type="fixed">
       <parent link="${parent}" />
@@ -220,9 +218,4 @@
       <origin xyz="0.0 -0.0335 0.0" rpy="${pi/2} 0 0" />
     </joint>
-    <joint name="${prefix}tcp_joint" type="fixed">
-      <parent link="${prefix}tool0_link" />
-      <child link="${prefix}tcp_link" />
-      <origin xyz="0.0 0.0 ${tcp_offset}" rpy="${-pi} 0 ${pi/2}" />
-    </joint>
   </xacro:macro>
 </robot>

Commit message: allow change max vel, acc, jerk in urdf macro

File: aubo_driver/urdf/aubo.ros2_control.xacro (robot description, xacro)
@@ -1,5 +1,14 @@
 <?xml version="1.0"?>
 <robot xmlns:xacro="http://www.ros.org/wiki/xacro">
-  <xacro:macro name="aubo_ros2_control" params="name prefix robot_ip use_mock_hardware:=false mock_sensor_commands:=false">
+  <xacro:macro name="aubo_ros2_control" params="
+   name
+   prefix
+   robot_ip
+   use_mock_hardware:=false
+   mock_sensor_commands:=false
+   max_vel_limit:=3.1
+   max_acc_limit:=6.0
+   max_jerk_limit:=20.0
+   ">
     <ros2_control name="${name}" type="system">
       <hardware>
@@ -16,10 +25,10 @@
           <param name="robot_ip">${robot_ip}</param>
           <param name="servoj_frequency">100</param>
-          <param name="servoj_smooth_scale">0.5</param>
-          <param name="servoj_delay_scale">0.5</param>
+          <param name="servoj_smooth_scale">1.0</param>
+          <param name="servoj_delay_scale">1.0</param>
           <param name="servoj_buffer_time">0.0</param>
-          <param name="max_vel_limit">3.1</param>
-          <param name="max_acc_limit">6.0</param>
-          <param name="max_jerk_limit">20.0</param>
+          <param name="max_vel_limit">${max_vel_limit}</param>
+          <param name="max_acc_limit">${max_acc_limit}</param>
+          <param name="max_jerk_limit">${max_jerk_limit}</param>
         </xacro:unless>
       </hardware>
